Commit message: add support for gazebo and gz using ros2 control

File: robots/robot.urdf.xacro (robot description, xacro)
@@ -1,15 +1,22 @@
 <?xml version="1.0" ?>
 <robot name="robot" xmlns:xacro="http://www.ros.org/wiki/xacro">
-    <xacro:include filename="./../urdf/skratch_base/skratch_top_base.urdf.xacro"/>
-    <xacro:include filename="./../urdf/skratch_base/skratch_bottom_base.urdf.xacro"/>
-    <xacro:include filename="./../urdf/skratch_base/skratch_wheel_support.urdf.xacro"/>
-    <xacro:include filename="./../urdf/skratch_wheels/skratch_wheel_hub.urdf.xacro"/>
-    <xacro:include filename="./../urdf/skratch_wheels/skratch_wheel.urdf.xacro"/>
-    <link name="base_link">
+    <xacro:include filename="$(find skratch_description)/urdf/skratch_base/skratch_top_base.urdf.xacro"/>
+    <xacro:include filename="$(find skratch_description)/urdf/skratch_base/skratch_bottom_base.urdf.xacro"/>
+    <xacro:include filename="$(find skratch_description)/urdf/skratch_base/skratch_wheel_support.urdf.xacro"/>
+    <xacro:include filename="$(find skratch_description)/urdf/skratch_wheels/skratch_wheel_hub.urdf.xacro"/>
+    <xacro:include filename="$(find skratch_description)/urdf/skratch_wheels/skratch_wheel.urdf.xacro"/>
+    <xacro:include filename="$(find skratch_description)/urdf/skratch_macro.ros2_control.xacro" />
+    <xacro:arg name="robot_name" default=""/>                   <!-- used by the launch system -->
+    <xacro:arg name="sim_gazebo" default="false"/>              <!-- used by the launch system (gazebo "classic")-->
+    <xacro:arg name="sim_gz" default="false"/>                  <!-- used by the launch system (latest version of gazebo) -->
+    <xacro:arg name="controllers" default=""/>                  <!-- used by the launch system -->
+    <xacro:property name="namespace" default="$(arg robot_name)"/>
+    <xacro:property name="prefix" default="${namespace}_" />
+    <link name="${prefix}base_link">
     </link>
     <xacro:skratch_top_base name="left_skratch_top_base"/>
     <joint name="base_joint" type="fixed">
         <origin xyz="0.0 -0.005 0.0" rpy="0.0 0.0 0.0"/>
-        <parent link="base_link"/>
+        <parent link="${prefix}base_link"/>
         <child link="left_skratch_top_base"/>
     </joint>
@@ -17,5 +24,5 @@
     <joint name="frame_joint" type="fixed">
         <origin xyz="0.0 0.003 0.0" rpy="0.0 0.0 3.14"/>
-        <parent link="base_link"/>
+        <parent link="${prefix}base_link"/>
         <child link="right_skratch_top_base"/>
     </joint>
@@ -128,3 +135,25 @@
         <axis xyz="0.0 1.0 0.0"/>
     </joint>
+    <xacro:if value="$(arg sim_gazebo)">
+        <xacro:macro_ros2_control name="GazeboSystem" plugin="gazebo_ros2_control/GazeboSystem"/>
+        <gazebo>
+            <plugin filename="libgazebo_ros2_control.so" name="gazebo_ros2_control">
+                <parameters>$(arg controllers)</parameters>
+                <ros>
+                    <namespace>${namespace}</namespace>
+                </ros>
+            </plugin>
+        </gazebo>
+    </xacro:if>
+    <xacro:if value="$(arg sim_gz)">
+        <xacro:macro_ros2_control name="IgnitionSystem" plugin="ign_ros2_control/IgnitionSystem"/>
+        <gazebo>
+            <plugin filename="ign_ros2_control-system" name="ign_ros2_control::IgnitionROS2ControlPlugin">
+                <parameters>$(arg controllers)</parameters>
+                <ros>
+                    <namespace>${namespace}</namespace>
+                </ros>
+            </plugin>
+        </gazebo>
+    </xacro:if>
 </robot>

Commit message: add support for imu gazebo classic

File: robots/robot.urdf.xacro (robot description, xacro)
@@ -7,4 +7,5 @@
     <xacro:include filename="$(find skratch_description)/urdf/skratch_wheels/skratch_wheel.urdf.xacro"/>
     <xacro:include filename="$(find skratch_description)/urdf/skratch_macro.ros2_control.xacro" />
+    <xacro:include filename="$(find skratch_description)/urdf/skratch_macro.imu_gazebo.xacro" />
     <xacro:arg name="robot_name" default=""/>                   <!-- used by the launch system -->
     <xacro:arg name="sim_gazebo" default="false"/>              <!-- used by the launch system (gazebo "classic")-->
@@ -15,51 +16,54 @@
     <link name="${prefix}base_link">
     </link>
-    <xacro:skratch_top_base name="left_skratch_top_base"/>
+    <xacro:skratch_top_base name="left_top_base"/>
     <joint name="base_joint" type="fixed">
         <origin xyz="0.0 -0.005 0.0" rpy="0.0 0.0 0.0"/>
         <parent link="${prefix}base_link"/>
-        <child link="left_skratch_top_base"/>
+        <child link="left_top_base"/>
     </joint>
-    <xacro:skratch_top_base name="right_skratch_top_base"/>
+    <xacro:skratch_top_base name="right_top_base"/>
     <joint name="frame_joint" type="fixed">
         <origin xyz="0.0 0.003 0.0" rpy="0.0 0.0 3.14"/>
         <parent link="${prefix}base_link"/>
-        <child link="right_skratch_top_base"/>
+        <child link="right_top_base"/>
     </joint>
-    <xacro:skratch_bottom_base name="left_skratch_bottom_base"/>
-    <joint name="left_skratch_bottom_base_joint" type="fixed">
+    <xacro:skratch_bottom_base name="left_bottom_base"/>
+    <joint name="left_bottom_base_joint" type="fixed">
         <origin xyz="0.0 -0.099 -0.138" rpy="3.14 0.0 0.0"/>
-        <parent link="left_skratch_top_base"/>
-        <child link="left_skratch_bottom_base"/>
+        <parent link="left_top_base"/>
+        <child link="left_bottom_base"/>
     </joint>
-    <xacro:skratch_bottom_base name="right_skratch_bottom_base"/>
-    <joint name="right_skratch_bottom_base_joint" type="fixed">
+    <xacro:skratch_bottom_base name="right_bottom_base"/>
+    <joint name="right_bottom_base_joint" type="fixed">
         <origin xyz="0.0 -0.099 -0.138" rpy="3.14 0.0 0.0"/>
-        <parent link="right_skratch_top_base"/>
-        <child link="right_skratch_bottom_base"/>
+        <parent link="right_top_base"/>
+        <child link="right_bottom_base"/>
     </joint>
-    <xacro:skratch_wheel_support name="left_skratch_wheel_support"/>
-    <joint name="left_skratch_wheel_support_joint" type="fixed">
+    <xacro:skratch_wheel_support name="left_wheel_support"/>
+    <joint name="left_wheel_support_joint" type="fixed">
         <origin xyz="0.0 0.0 -0.1022" rpy="0.0 0.0 0.0"/>
-        <parent link="left_skratch_bottom_base"/>
-        <child link="left_skratch_wheel_support"/>
+        <parent link="left_bottom_base"/>
+        <child link="left_wheel_support"/>
     </joint>
-    <xacro:skratch_wheel_support name="right_skratch_wheel_support"/>
-    <joint name="right_skratch_wheel_support_joint" type="fixed">
+    <xacro:skratch_wheel_support name="right_wheel_support"/>
+    <joint name="right_wheel_support_joint" type="fixed">
         <origin xyz="0.0 0.0 -0.1022" rpy="0.0 0.0 0.0"/>
-        <parent link="right_skratch_bottom_base"/>
-        <child link="right_skratch_wheel_support"/>
+        <parent link="right_bottom_base"/>
+        <child link="right_wheel_support"/>
     </joint>
-    <xacro:skratch_wheel_hub name="front_left_skratch_wheel_hub"/>
-    <joint name="front_left_skratch_wheel_hub_joint" type="continuous">
+    <xacro:skratch_wheel_hub name="front_left_wheel_hub"/>
+    <joint name="front_left_wheel_hub_joint" type="continuous">
         <origin xyz="0.2 0.0 0.085" rpy="3.14 0.0 0.0"/>
-        <parent link="left_skratch_wheel_support"/>
-        <child link="front_left_skratch_wheel_hub"/>
+        <parent link="left_wheel_support"/>
+        <child link="front_left_wheel_hub"/>
         <axis xyz="0.0 0.0 1.0"/>
     </joint>
+    <xacro:if value="$(arg sim_gazebo)">
+        <xacro:macro_imu_gazebo name="front_left_wheel_imu" parent_link="front_left_wheel_hub" namespace="${namespace}" />
+    </xacro:if>
     <xacro:skratch_wheel name="front_left_wheel_one"/>
     <joint name="front_left_wheel_one_joint" type="continuous">
         <origin xyz="0.0 0.04 0.0" rpy="0.0 0.0 0.0"/>
-        <parent link="front_left_skratch_wheel_hub"/>
+        <parent link="front_left_wheel_hub"/>
         <child link="front_left_wheel_one"/>
         <axis xyz="0.0 1.0 0.0"/>
@@ -68,19 +72,22 @@
     <joint name="front_left_wheel_two_joint" type="continuous">
         <origin xyz="0.0 -0.04 0.0" rpy="0.0 0.0 0.0"/>
-        <parent link="front_left_skratch_wheel_hub"/>
+        <parent link="front_left_wheel_hub"/>
         <child link="front_left_wheel_two"/>
         <axis xyz="0.0 1.0 0.0"/>
     </joint>
-    <xacro:skratch_wheel_hub name="front_right_skratch_wheel_hub"/>
-    <joint name="front_right_skratch_wheel_hub_joint" type="continuous">
+    <xacro:skratch_wheel_hub name="front_right_wheel_hub"/>
+    <joint name="front_right_wheel_hub_joint" type="continuous">
         <origin xyz="-0.2 0.0 0.085" rpy="3.14 0.0 0.0"/>
-        <parent link="right_skratch_wheel_support"/>
-        <child link="front_right_skratch_wheel_hub"/>
+        <parent link="right_wheel_support"/>
+        <child link="front_right_wheel_hub"/>
         <axis xyz="0.0 0.0 1.0"/>
     </joint>
+    <xacro:if value="$(arg sim_gazebo)">
+        <xacro:macro_imu_gazebo name="front_right_wheel_imu" parent_link="front_right_wheel_hub" namespace="${namespace}" />
+    </xacro:if>
     <xacro:skratch_wheel name="front_right_wheel_one"/>
     <joint name="front_right_wheel_one_joint" type="continuous">
         <origin xyz="0.0 0.04 0.0" rpy="0.0 0.0 0.0"/>
-        <parent link="front_right_skratch_wheel_hub"/>
+        <parent link="front_right_wheel_hub"/>
         <child link="front_right_wheel_one"/>
         <axis xyz="0.0 1.0 0.0"/>
@@ -89,19 +96,22 @@
     <joint name="front_right_wheel_two_joint" type="continuous">
         <origin xyz="0.0 -0.04 0.0" rpy="0.0 0.0 0.0"/>
-        <parent link="front_right_skratch_wheel_hub"/>
+        <parent link="front_right_wheel_hub"/>
         <child link="front_right_wheel_two"/>
         <axis xyz="0.0 1.0 0.0"/>
     </joint>
-    <xacro:skratch_wheel_hub name="rear_left_skratch_wheel_hub"/>
-    <joint name="rear_left_skratch_wheel_hub_joint" type="continuous">
+    <xacro:skratch_wheel_hub name="rear_left_wheel_hub"/>
+    <joint name="rear_left_wheel_hub_joint" type="continuous">
         <origin xyz="-0.2 0.0 0.085" rpy="3.14 0.0 0.0"/>
-        <parent link="left_skratch_wheel_support"/>
-        <child link="rear_left_skratch_wheel_hub"/>
+        <parent link="left_wheel_support"/>
+        <child link="rear_left_wheel_hub"/>
         <axis xyz="0.0 0.0 1.0"/>
     </joint>
+    <xacro:if value="$(arg sim_gazebo)">
+        <xacro:macro_imu_gazebo name="rear_left_wheel_imu" parent_link="rear_left_wheel_hub" namespace="${namespace}" />
+    </xacro:if>
     <xacro:skratch_wheel name="rear_left_wheel_one"/>
     <joint name="rear_left_wheel_one_joint" type="continuous">
         <origin xyz="0.0 0.04 0.0" rpy="0.0 0.0 0.0"/>
-        <parent link="rear_left_skratch_wheel_hub"/>
+        <parent link="rear_left_wheel_hub"/>
         <child link="rear_left_wheel_one"/>
         <axis xyz="0.0 1.0 0.0"/>
@@ -110,19 +120,22 @@
     <joint name="rear_left_wheel_two_joint" type="continuous">
         <origin xyz="0.0 -0.04 0.0" rpy="0.0 0.0 0.0"/>
-        <parent link="rear_left_skratch_wheel_hub"/>
+        <parent link="rear_left_wheel_hub"/>
         <child link="rear_left_wheel_two"/>
         <axis xyz="0.0 1.0 0.0"/>
     </joint>
-    <xacro:skratch_wheel_hub name="rear_right_skratch_wheel_hub"/>
-    <joint name="rear_right_skratch_wheel_hub_joint" type="continuous">
+    <xacro:skratch_wheel_hub name="rear_right_wheel_hub"/>
+    <joint name="rear_right_wheel_hub_joint" type="continuous">
         <origin xyz="0.2 0.0 0.085" rpy="3.14 0.0 0.0"/>
-        <parent link="right_skratch_wheel_support"/>
-        <child link="rear_right_skratch_wheel_hub"/>
+        <parent link="right_wheel_support"/>
+        <child link="rear_right_wheel_hub"/>
         <axis xyz="0.0 0.0 1.0"/>
     </joint>
+    <xacro:if value="$(arg sim_gazebo)">
+        <xacro:macro_imu_gazebo name="rear_right_wheel_imu" parent_link="rear_right_wheel_hub" namespace="${namespace}" />
+    </xacro:if>
     <xacro:skratch_wheel name="rear_right_wheel_one"/>
     <joint name="rear_right_wheel_one_joint" type="continuous">
         <origin xyz="0.0 0.04 0.0" rpy="0.0 0.0 0.0"/>
-        <parent link="rear_right_skratch_wheel_hub"/>
+        <parent link="rear_right_wheel_hub"/>
         <child link="rear_right_wheel_one"/>
         <axis xyz="0.0 1.0 0.0"/>
@@ -131,5 +144,5 @@
     <joint name="rear_right_wheel_two_joint" type="continuous">
         <origin xyz="0.0 -0.04 0.0" rpy="0.0 0.0 0.0"/>
-        <parent link="rear_right_skratch_wheel_hub"/>
+        <parent link="rear_right_wheel_hub"/>
         <child link="rear_right_wheel_two"/>
         <axis xyz="0.0 1.0 0.0"/>

File: urdf/skratch_macro.ros2_control.xacro (robot description, xacro)
@@ -1,58 +1,106 @@
 <?xml version="1.0"?>
 <robot xmlns:xacro="http://www.ros.org/wiki/xacro">
-    <xacro:macro name="macro_ros2_control" params="name plugin">
-        <ros2_control name="${name}" type="system">
-            <hardware>
-                <plugin>${plugin}</plugin>
-            </hardware>
-            <joint name="rear_left_skratch_wheel_hub_joint">
-                <state_interface name="position"/>
-                <state_interface name="velocity"/>
-            </joint>
-            <joint name="rear_left_wheel_one_joint">
-                <state_interface name="position"/>
-                <state_interface name="velocity"/>
-            </joint>
-            <joint name="rear_left_wheel_two_joint">
-                <state_interface name="position"/>
-                <state_interface name="velocity"/>
-            </joint>
-            <joint name="rear_right_skratch_wheel_hub_joint">
-                <state_interface name="position"/>
-                <state_interface name="velocity"/>
-            </joint>
-            <joint name="rear_right_wheel_one_joint">
-                <state_interface name="position"/>
-                <state_interface name="velocity"/>
-            </joint>
-            <joint name="rear_right_wheel_two_joint">
-                <state_interface name="position"/>
-                <state_interface name="velocity"/>
-            </joint>
-            <joint name="front_left_skratch_wheel_hub_joint">
-                <state_interface name="position"/>
-                <state_interface name="velocity"/>
-            </joint>
-            <joint name="front_left_wheel_one_joint">
-                <state_interface name="position"/>
-                <state_interface name="velocity"/>
-            </joint>
-            <joint name="front_left_wheel_two_joint">
-                <state_interface name="position"/>
-                <state_interface name="velocity"/>
-            </joint>
-            <joint name="front_right_skratch_wheel_hub_joint">
-                <state_interface name="position"/>
-                <state_interface name="velocity"/>
-            </joint>
-            <joint name="front_right_wheel_one_joint">
-                <state_interface name="position"/>
-                <state_interface name="velocity"/>
-            </joint>
-            <joint name="front_right_wheel_two_joint">
-                <state_interface name="position"/>
-                <state_interface name="velocity"/>
-            </joint>
-        </ros2_control>
+  <xacro:macro name="macro_ros2_control" params="name plugin">
+    <ros2_control name="${name}" type="system">
+      <hardware>
+        <plugin>${plugin}</plugin>
+        </hardware>
+      <sensor name="front_left_wheel_imu">
+        <state_interface name="orientation.x"/>
+        <state_interface name="orientation.y"/>
+        <state_interface name="orientation.z"/>
+        <state_interface name="orientation.w"/>
+        <state_interface name="angular_velocity.x"/>
+        <state_interface name="angular_velocity.y"/>
+        <state_interface name="angular_velocity.z"/>
+        <state_interface name="linear_acceleration.x"/>
+        <state_interface name="linear_acceleration.y"/>
+        <state_interface name="linear_acceleration.z"/>
+        </sensor>
+      <sensor name="front_right_wheel_imu">
+        <state_interface name="orientation.x"/>
+        <state_interface name="orientation.y"/>
+        <state_interface name="orientation.z"/>
+        <state_interface name="orientation.w"/>
+        <state_interface name="angular_velocity.x"/>
+        <state_interface name="angular_velocity.y"/>
+        <state_interface name="angular_velocity.z"/>
+        <state_interface name="linear_acceleration.x"/>
+        <state_interface name="linear_acceleration.y"/>
+        <state_interface name="linear_acceleration.z"/>
+        </sensor>
+      <sensor name="rear_left_wheel_imu">
+        <state_interface name="orientation.x"/>
+        <state_interface name="orientation.y"/>
+        <state_interface name="orientation.z"/>
+        <state_interface name="orientation.w"/>
+        <state_interface name="angular_velocity.x"/>
+        <state_interface name="angular_velocity.y"/>
+        <state_interface name="angular_velocity.z"/>
+        <state_interface name="linear_acceleration.x"/>
+        <state_interface name="linear_acceleration.y"/>
+        <state_interface name="linear_acceleration.z"/>
+        </sensor>
+      <sensor name="rear_right_wheel_imu">
+        <state_interface name="orientation.x"/>
+        <state_interface name="orientation.y"/>
+        <state_interface name="orientation.z"/>
+        <state_interface name="orientation.w"/>
+        <state_interface name="angular_velocity.x"/>
+        <state_interface name="angular_velocity.y"/>
+        <state_interface name="angular_velocity.z"/>
+        <state_interface name="linear_acceleration.x"/>
+        <state_interface name="linear_acceleration.y"/>
+        <state_interface name="linear_acceleration.z"/>
+        </sensor>
+      <joint name="rear_left_wheel_hub_joint">
+        <state_interface name="position"/>
+        <state_interface name="velocity"/>
+        </joint>
+      <joint name="rear_left_wheel_one_joint">
+        <state_interface name="position"/>
+        <state_interface name="velocity"/>
+        </joint>
+      <joint name="rear_left_wheel_two_joint">
+        <state_interface name="position"/>
+        <state_interface name="velocity"/>
+        </joint>
+      <joint name="rear_right_wheel_hub_joint">
+        <state_interface name="position"/>
+        <state_interface name="velocity"/>
+        </joint>
+      <joint name="rear_right_wheel_one_joint">
+        <state_interface name="position"/>
+        <state_interface name="velocity"/>
+        </joint>
+      <joint name="rear_right_wheel_two_joint">
+        <state_interface name="position"/>
+        <state_interface name="velocity"/>
+        </joint>
+      <joint name="front_left_wheel_hub_joint">
+        <state_interface name="position"/>
+        <state_interface name="velocity"/>
+        </joint>
+      <joint name="front_left_wheel_one_joint">
+        <state_interface name="position"/>
+        <state_interface name="velocity"/>
+        </joint>
+      <joint name="front_left_wheel_two_joint">
+        <state_interface name="position"/>
+        <state_interface name="velocity"/>
+        </joint>
+      <joint name="front_right_wheel_hub_joint">
+        <state_interface name="position"/>
+        <state_interface name="velocity"/>
+        </joint>
+      <joint name="front_right_wheel_one_joint">
+        <state_interface name="position"/>
+        <state_interface name="velocity"/>
+        </joint>
+      <joint name="front_right_wheel_two_joint">
+        <state_interface name="position"/>
+        <state_interface name="velocity"/>
+        </joint>
+      </ros2_control>
     </xacro:macro>
-</robot>
+  </robot>
