Commit message: add imu support for gazebo fortress

File: robots/robot.urdf.xacro (robot description, xacro)
@@ -8,4 +8,5 @@
     <xacro:include filename="$(find skratch_description)/urdf/skratch_macro.ros2_control.xacro" />
     <xacro:include filename="$(find skratch_description)/urdf/skratch_macro.imu_gazebo.xacro" />
+    <xacro:include filename="$(find skratch_description)/urdf/skratch_macro.imu_gz.xacro" />
     <xacro:arg name="robot_name" default=""/>                   <!-- used by the launch system -->
     <xacro:arg name="sim_gazebo" default="false"/>              <!-- used by the launch system (gazebo "classic")-->
@@ -62,4 +63,7 @@
         <xacro:macro_imu_gazebo name="front_left_wheel_imu" parent_link="front_left_wheel_hub" namespace="${namespace}" />
     </xacro:if>
+    <xacro:if value="$(arg sim_gz)">
+        <xacro:macro_imu_gz name="front_left_wheel_imu" parent_link="front_left_wheel_hub" namespace="${namespace}" />
+    </xacro:if>
     <xacro:skratch_wheel name="front_left_wheel_one"/>
     <joint name="front_left_wheel_one_joint" type="continuous">
@@ -85,4 +89,7 @@
     <xacro:if value="$(arg sim_gazebo)">
         <xacro:macro_imu_gazebo name="front_right_wheel_imu" parent_link="front_right_wheel_hub" namespace="${namespace}" />
+    </xacro:if>
+    <xacro:if value="$(arg sim_gz)">
+        <xacro:macro_imu_gz name="front_right_wheel_imu" parent_link="front_right_wheel_hub" namespace="${namespace}" />
     </xacro:if>
     <xacro:skratch_wheel name="front_right_wheel_one"/>
@@ -110,4 +117,7 @@
         <xacro:macro_imu_gazebo name="rear_left_wheel_imu" parent_link="rear_left_wheel_hub" namespace="${namespace}" />
     </xacro:if>
+    <xacro:if value="$(arg sim_gz)">
+        <xacro:macro_imu_gz name="rear_left_wheel_imu" parent_link="rear_left_wheel_hub" namespace="${namespace}" />
+    </xacro:if>
     <xacro:skratch_wheel name="rear_left_wheel_one"/>
     <joint name="rear_left_wheel_one_joint" type="continuous">
@@ -132,5 +142,8 @@
     </joint>
     <xacro:if value="$(arg sim_gazebo)">
-        <xacro:macro_imu_gazebo name="rear_right_wheel_imu" parent_link="rear_right_wheel_hub" namespace="${namespace}" />
+        <xacro:macro_imu_gz name="rear_right_wheel_imu" parent_link="rear_right_wheel_hub" namespace="${namespace}" />
+    </xacro:if>
+    <xacro:if value="$(arg sim_gz)">
+        <xacro:macro_imu_gz name="rear_right_wheel_imu" parent_link="rear_right_wheel_hub" namespace="${namespace}" />
     </xacro:if>
     <xacro:skratch_wheel name="rear_right_wheel_one"/>

File: urdf/skratch_macro.imu_gazebo.xacro (robot description, xacro)
@@ -1,16 +1,9 @@
 <?xml version="1.0"?>
 <robot xmlns:xacro="http://www.ros.org/wiki/xacro">
+  <xacro:include filename="$(find skratch_description)/urdf/skratch_macro.imu.xacro" />
   <xacro:macro name="macro_imu_gazebo" params="name parent_link namespace">
-    <link name="${name}_link">
-      <inertial>
-        <mass value="0.1"/>
-        <inertia ixx="1.0" ixy="0" ixz="0" iyy="1.0" iyz="0" izz="1.0"/>
-        </inertial>
-      </link>
-    <joint name="${name}_joint" type="fixed">
-      <parent link="${parent_link}"/>
-      <child link="${name}_link"/>
-      <origin xyz="0 0 0"/>
-      </joint>
+    <xacro:imu name="${name}" parent_link="${parent_link}" />
+    <!-- The Offical documentation for IMU on Gazebo "Classic" -->
+    <!-- check: https://classic.gazebosim.org/tutorials?tut=ros_gzplugins -->
     <gazebo reference="${name}_link"> <!-- IMPORTANT!  it needs to be the same as the link name -->
       <gravity>true</gravity>
