Commit message: fix Parser Error Couldn't parse parameter override rule, see https://github.com/ros-controls/gazebo_ros2_control/issues/295#issuecomment-2024692482

File: urdf/skratch_macro.imu.xacro (robot description, xacro)
@@ -5,5 +5,5 @@
       <inertial>
         <mass value="0.01"/>
-        <inertia ixx="1.0" ixy="0" ixz="0" iyy="1.0" iyz="0" izz="1.0"/> <!--TODO: set more realistic values -->
+        <inertia ixx="1.0" ixy="0" ixz="0" iyy="1.0" iyz="0" izz="1.0"/>
         </inertial>
     </link>

File: urdf/skratch_macro.imu_gazebo.xacro (robot description, xacro)
@@ -4,6 +4,4 @@
   <xacro:macro name="macro_imu_gazebo" params="name parent_link namespace">
     <xacro:imu name="${name}" parent_link="${parent_link}" />
-    <!-- The Offical documentation for IMU on Gazebo "Classic" -->
-    <!-- check: https://classic.gazebosim.org/tutorials?tut=ros_gzplugins -->
     <gazebo reference="${name}_link"> <!-- IMPORTANT!  it needs to be the same as the link name -->
       <gravity>true</gravity>

File: urdf/skratch_macro.imu_gz.xacro (robot description, xacro)
@@ -4,6 +4,4 @@
   <xacro:macro name="macro_imu_gz" params="name parent_link namespace">
     <xacro:imu name="${name}" parent_link="${parent_link}" />
-    <!-- For details on IMU sensor on gazebo "gz"-->
-    <!-- See: https://gazebosim.org/docs/fortress/sensors/#imu-sensor -->
     <gazebo reference="${name}_link"> <!-- IMPORTANT!  it needs to be the same as the link name -->
       <gravity>true</gravity>
