Commit message: add textures to wheels

File: urdf/skratch_wheels/skratch_wheel.urdf.xacro (robot description, xacro)
@@ -11,5 +11,5 @@
                 <origin xyz="0.0 0.0 0.0" rpy="0.0 0.0 0.0" />
                 <geometry>
-                    <mesh filename="file://$(find skratch_description)/meshes/skratch_wheel/kelo_drive_wheel.stl" scale="1 1 1"/>
+                    <mesh filename="file://$(find skratch_description)/meshes/skratch_wheel/kelo_drive_wheel.dae" scale="1 1 1"/>
                 </geometry>
             </visual>
@@ -17,5 +17,5 @@
                 <origin xyz="0.0 0.0 0.0" rpy="0.0 0.0 0.0" />
                 <geometry>
-                    <mesh filename="file://$(find skratch_description)/meshes/skratch_wheel/kelo_drive_wheel.stl" scale="1 1 1"/>
+                    <mesh filename="file://$(find skratch_description)/meshes/skratch_wheel/kelo_drive_wheel.dae" scale="1 1 1"/>
                 </geometry>
             </collision>

File: urdf/skratch_wheels/skratch_wheel_hub.urdf.xacro (robot description, xacro)
@@ -11,5 +11,5 @@
                 <origin xyz="0.0 0.0 0.0" rpy="0.0 0.0 0.0" />
                 <geometry>
-                    <mesh filename="file://$(find skratch_description)/meshes/skratch_wheel/kelo_drive_base.stl" scale="1 1 1"/>
+                    <mesh filename="file://$(find skratch_description)/meshes/skratch_wheel/kelo_drive_base.dae" scale="1 1 1"/>
                 </geometry>
             </visual>
@@ -17,5 +17,5 @@
                 <origin xyz="0.0 0.0 0.0" rpy="0.0 0.0 0.0" />
                 <geometry>
-                    <mesh filename="file://$(find skratch_description)/meshes/skratch_wheel/kelo_drive_base.stl" scale="1 1 1"/>
+                    <mesh filename="file://$(find skratch_description)/meshes/skratch_wheel/kelo_drive_base.dae" scale="1 1 1"/>
                 </geometry>
             </collision>
