Commit message: fix mesh file URI to fully resolve path (for gazebo)

File: urdf/skratch_base/skratch_bottom_base.urdf.xacro (robot description, xacro)
@@ -11,5 +11,5 @@
                 <origin xyz="0.0 0.0 0.0" rpy="0.0 0.0 0.0" />
                 <geometry>
-                    <mesh filename="package://skratch_description/meshes/skratch_base/skratch_bottom_base.stl" scale="0.001 0.001 0.001"/>
+                    <mesh filename="file://$(find skratch_description)/meshes/skratch_base/skratch_bottom_base.stl" scale="0.001 0.001 0.001"/>
                 </geometry>
             </visual>
@@ -17,5 +17,5 @@
                 <origin xyz="0.0 0.0 0.0" rpy="0.0 0.0 0.0" />
                 <geometry>
-                    <mesh filename="package://skratch_description/meshes/skratch_base/skratch_bottom_base.stl" scale="0.001 0.001 0.001"/>
+                    <mesh filename="file://$(find skratch_description)/meshes/skratch_base/skratch_bottom_base.stl" scale="0.001 0.001 0.001"/>
                 </geometry>
             </collision>

File: urdf/skratch_base/skratch_top_base.urdf.xacro (robot description, xacro)
@@ -11,5 +11,5 @@
                 <origin xyz="0.0 0.0 0.0" rpy="0.0 0.0 0.0" />
                 <geometry>
-                    <mesh filename="package://skratch_description/meshes/skratch_base/skratch_top_base.stl" scale="0.001 0.001 0.001"/>
+                    <mesh filename="file://$(find skratch_description)/meshes/skratch_base/skratch_top_base.stl" scale="0.001 0.001 0.001"/>
                 </geometry>
             </visual>
@@ -17,5 +17,5 @@
                 <origin xyz="0.0 0.0 0.0" rpy="0.0 0.0 0.0" />
                 <geometry>
-                    <mesh filename="package://skratch_description/meshes/skratch_base/skratch_top_base.stl" scale="0.001 0.001 0.001"/>
+                    <mesh filename="file://$(find skratch_description)/meshes/skratch_base/skratch_top_base.stl" scale="0.001 0.001 0.001"/>
                 </geometry>
             </collision>

File: urdf/skratch_base/skratch_wheel_support.urdf.xacro (robot description, xacro)
@@ -11,5 +11,5 @@
                 <origin xyz="0.0 0.0 0.0" rpy="0.0 0.0 0.0" />
                 <geometry>
-                    <mesh filename="package://skratch_description/meshes/skratch_base/skratch_wheel_support.stl" scale="0.001 0.001 0.001"/>
+                    <mesh filename="file://$(find skratch_description)/meshes/skratch_base/skratch_wheel_support.stl" scale="0.001 0.001 0.001"/>
                 </geometry>
             </visual>
@@ -17,5 +17,5 @@
                 <origin xyz="0.0 0.0 0.0" rpy="0.0 0.0 0.0" />
                 <geometry>
-                    <mesh filename="package://skratch_description/meshes/skratch_base/skratch_wheel_support.stl" scale="0.001 0.001 0.001"/>
+                    <mesh filename="file://$(find skratch_description)/meshes/skratch_base/skratch_wheel_support.stl" scale="0.001 0.001 0.001"/>
                 </geometry>
             </collision>

File: urdf/skratch_wheels/skratch_wheel.urdf.xacro (robot description, xacro)
@@ -11,5 +11,5 @@
                 <origin xyz="0.0 0.0 0.0" rpy="0.0 0.0 0.0" />
                 <geometry>
-                    <mesh filename="package://skratch_description/meshes/skratch_wheel/kelo_drive_wheel.stl" scale="1 1 1"/>
+                    <mesh filename="file://$(find skratch_description)/meshes/skratch_wheel/kelo_drive_wheel.stl" scale="1 1 1"/>
                 </geometry>
             </visual>
@@ -17,5 +17,5 @@
                 <origin xyz="0.0 0.0 0.0" rpy="0.0 0.0 0.0" />
                 <geometry>
-                    <mesh filename="package://skratch_description/meshes/skratch_wheel/kelo_drive_wheel.stl" scale="1 1 1"/>
+                    <mesh filename="file://$(find skratch_description)/meshes/skratch_wheel/kelo_drive_wheel.stl" scale="1 1 1"/>
                 </geometry>
             </collision>

File: urdf/skratch_wheels/skratch_wheel_hub.urdf.xacro (robot description, xacro)
@@ -11,5 +11,5 @@
                 <origin xyz="0.0 0.0 0.0" rpy="0.0 0.0 0.0" />
                 <geometry>
-                    <mesh filename="package://skratch_description/meshes/skratch_wheel/kelo_drive_base.stl" scale="1 1 1"/>
+                    <mesh filename="file://$(find skratch_description)/meshes/skratch_wheel/kelo_drive_base.stl" scale="1 1 1"/>
                 </geometry>
             </visual>
@@ -17,5 +17,5 @@
                 <origin xyz="0.0 0.0 0.0" rpy="0.0 0.0 0.0" />
                 <geometry>
-                    <mesh filename="package://skratch_description/meshes/skratch_wheel/kelo_drive_base.stl" scale="1 1 1"/>
+                    <mesh filename="file://$(find skratch_description)/meshes/skratch_wheel/kelo_drive_base.stl" scale="1 1 1"/>
                 </geometry>
             </collision>

Commit message: add mesh with textures

File: urdf/skratch_base/skratch_bottom_base.urdf.xacro (robot description, xacro)
@@ -11,5 +11,5 @@
                 <origin xyz="0.0 0.0 0.0" rpy="0.0 0.0 0.0" />
                 <geometry>
-                    <mesh filename="file://$(find skratch_description)/meshes/skratch_base/skratch_bottom_base.stl" scale="0.001 0.001 0.001"/>
+                    <mesh filename="file://$(find skratch_description)/meshes/skratch_base/skratch_bottom_base.dae" scale="1 1 1"/>
                 </geometry>
             </visual>
@@ -17,5 +17,5 @@
                 <origin xyz="0.0 0.0 0.0" rpy="0.0 0.0 0.0" />
                 <geometry>
-                    <mesh filename="file://$(find skratch_description)/meshes/skratch_base/skratch_bottom_base.stl" scale="0.001 0.001 0.001"/>
+                    <mesh filename="file://$(find skratch_description)/meshes/skratch_base/skratch_bottom_base.dae" scale="1 1 1"/>
                 </geometry>
             </collision>

File: urdf/skratch_base/skratch_top_base.urdf.xacro (robot description, xacro)
@@ -11,5 +11,5 @@
                 <origin xyz="0.0 0.0 0.0" rpy="0.0 0.0 0.0" />
                 <geometry>
-                    <mesh filename="file://$(find skratch_description)/meshes/skratch_base/skratch_top_base.stl" scale="0.001 0.001 0.001"/>
+                    <mesh filename="file://$(find skratch_description)/meshes/skratch_base/skratch_top_base.dae" scale="1 1 1"/>
                 </geometry>
             </visual>
@@ -17,5 +17,5 @@
                 <origin xyz="0.0 0.0 0.0" rpy="0.0 0.0 0.0" />
                 <geometry>
-                    <mesh filename="file://$(find skratch_description)/meshes/skratch_base/skratch_top_base.stl" scale="0.001 0.001 0.001"/>
+                    <mesh filename="file://$(find skratch_description)/meshes/skratch_base/skratch_top_base.dae" scale="1 1 1"/>
                 </geometry>
             </collision>

File: urdf/skratch_base/skratch_wheel_support.urdf.xacro (robot description, xacro)
@@ -11,5 +11,5 @@
                 <origin xyz="0.0 0.0 0.0" rpy="0.0 0.0 0.0" />
                 <geometry>
-                    <mesh filename="file://$(find skratch_description)/meshes/skratch_base/skratch_wheel_support.stl" scale="0.001 0.001 0.001"/>
+                    <mesh filename="file://$(find skratch_description)/meshes/skratch_base/skratch_wheel_support.dae" scale="1 1 1"/>
                 </geometry>
             </visual>
@@ -17,5 +17,5 @@
                 <origin xyz="0.0 0.0 0.0" rpy="0.0 0.0 0.0" />
                 <geometry>
-                    <mesh filename="file://$(find skratch_description)/meshes/skratch_base/skratch_wheel_support.stl" scale="0.001 0.001 0.001"/>
+                    <mesh filename="file://$(find skratch_description)/meshes/skratch_base/skratch_wheel_support.dae" scale="1 1 1"/>
                 </geometry>
             </collision>
